File: Lectures/03/led_and_resistor_board.kicad_pcb (KiCad board)
At the start: 2 copper layers, 59.7 x 17.8 mm, 4 parts

Commit message: Terminal Block
Parts:
- removed the REF** at (180.3, 99.1)
- added J1: Conn_01x02_Male, TerminalBlock:TerminalBlock_bornier-2_P5.08mm, F.Cu at (180.3, 99.1)
Routing:
- net GND: track 34.7 -> 41.9 mm
- net (no net): track 7.18 -> 0.00 mm
